File: heated_bed/.kicad_pcb.kicad_pcb (KiCad board)
At the start: 2 copper layers, 220 x 215 mm, 10 parts, among them P1 CONN_4

Commit message: Placa assinada
Routing:
- net (no net): track 18.0 -> 0.00 mm
Changed lines of the file:
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@@
     (thickness 1.6)
     (drawings 23)
-    (tracks 931)
+    (tracks 910)
     (zones 0)
     (modules 10)
@@
   (gr_line (start 244 18) (end 244 233) (angle 90) (layer Edge.Cuts) (width 0.15))
   (gr_line (start 24 18) (end 244 18) (angle 90) (layer Edge.Cuts) (width 0.15))
-  (segment (start 34 23.5) (end 34 24) (width 0.254) (layer B.Cu) (net 0))
-  (segment (start 33.5 23.5) (end 34 23.5) (width 0.254) (layer B.Cu) (net 0))
-  (segment (start 31 26) (end 31 26.5) (width 0.254) (layer B.Cu) (net 0))
-  (segment (start 30.5 26) (end 31 26) (width 0.254) (layer B.Cu) (net 0))
-  (segment (start 33 25.5) (end 34.5 27) (width 0.254) (layer B.Cu) (net 0))
-  (segment (start 33 24.5) (end 33.5 24) (width 0.254) (layer B.Cu) (net 0))
-  (segment (start 33.5 24) (end 34 23.5) (width 0.254) (layer B.Cu) (net 0))
-  (segment (start 34 23.5) (end 34.5 23) (width 0.254) (layer B.Cu) (net 0))
-  (segment (start 31.5 25.5) (end 31 26) (width 0.254) (layer B.Cu) (net 0))
-  (segment (start 31 26) (end 30.5 26.5) (width 0.254) (layer B.Cu) (net 0))
-  (segment (start 30.5 26.5) (end 30 27) (width 0.254) (layer B.Cu) (net 0))
-  (segment (start 30 23) (end 31.5 24.5) (width 0.254) (layer B.Cu) (net 0))
-  (segment (start 31.5 25) (end 33 25) (width 0.254) (layer B.Cu) (net 0))
-  (segment (start 33 23.5) (end 33 24.5) (width 0.254) (layer B.Cu) (net 0))
-  (segment (start 33 24.5) (end 33 25) (width 0.254) (layer B.Cu) (net 0))
-  (segment (start 33 25) (end 33 25.5) (width 0.254) (layer B.Cu) (net 0))
-  (segment (start 33 25.5) (end 33 26.5) (width 0.254) (layer B.Cu) (net 0))
-  (segment (start 31.5 23.5) (end 31.5 24.5) (width 0.254) (layer B.Cu) (net 0))
-  (segment (start 31.5 24.5) (end 31.5 25) (width 0.254) (layer B.Cu) (net 0))
-  (segment (start 31.5 25) (end 31.5 25.5) (width 0.254) (layer B.Cu) (net 0))
-  (segment (start 31.5 25.5) (end 31.5 26.5) (width 0.254) (layer B.Cu) (net 0))
   (segment (start 142.5 126.262) (end 140.6905 126.262) (width 0.254) (layer B.Cu) (net 1))
   (segment (start 140.6905 126.262) (end 140.5 126.4525) (width 0.254) (layer B.Cu) (net 1))
